File: redline_v3/redline_v3.kicad_sch (KiCad schematic)
At the start: 67 parts, among them J1 Conn_01x10_Socket, J2 Conn_01x10_Socket

Commit message: traces all done
Parts:
- removed J1, J2: Conn_01x10_Socket, Connector_PinSocket_1.00mm:PinSocket_1x10_P1.00mm_Vertical, symbol Connector:Conn_01x10_Socket
- added C1: 10nF, Capacitor_SMD:C_0603_1608Metric, symbol Device:C
- added C2: 3.3nF, Capacitor_SMD:C_0603_1608Metric, symbol Device:C
- added C3, C4: C_1uF, footprints:C_0603_1608Metric, symbol formula:C_1uF
- added J4: 48037-0001, custom_library:MOLEX_USB_conn, symbol usb_conn:48037-0001
- added R8: R_US, Resistor_SMD:R_0603_1608Metric, symbol Device:R_US
- added U1: ESP32, Package_DFN_QFN:QFN-48-1EP_8x8mm_P0.5mm_EP6.2x6.2mm, symbol PCM_Espressif:ESP32
- added U2: MCP1702T-3302E_MB, custom_library:MCP1702T, symbol LDO_MCP1702T-3302E_MB:MCP1702T-3302E_MB
Connections:
- net 0: now also U1.14 (GPIO25/ADC2_CH8/DAC_1)
- net 1: now also U1.15 (GPIO26/ADC2_CH9/DAC_2)
- net 2: now also U1.16 (GPIO27/ADC2_CH7)
- net 3: now also U1.31 (SD_CLK/GPIO6)
- net 4: now also U1.32 (SD_DATA_0/GPIO7)
- net 5: now also U1.33 (SD_DATA_1/GPIO8)
- net 6: now also U1.28 (SD_DATA_2/GPIO9)
- net 7: now also U1.29 (SD_DATA_3/GPIO10)
- net 8: now also U1.30 (SD_CMD/GPIO11)
- net 9: now also U1.25 (GPIO16)
- net A: now also U1.24 (GPIO4/ADC2_CH0)
- net B: now also U1.34 (GPIO5)
- net C: now also U1.35 (GPIO18)
- net D: now also U1.38 (GPIO19)
- net E: now also U1.42 (GPIO21)
- net F: now also U1.39 (GPIO22)
- net G: now also U1.36 (GPIO23)
- net GND: now also C1.2, C2.1, C3.2, C4.2, J4.4 (GND), U1.49 (GND), U2.1 (GND)
- new net: U1.3 (VDD3P3), U1.4 (VDD3P3)
- new net: C1.1, R8.2, U1.47 (CAP2), U1.48 (CAP1)
- new net: C3.1, J4.1 (VCC), U2.2 (VIN)
- new net: C2.2, R8.1
- new net +3.3V: C4.1, U1.1 (VDDA), U1.37 (VDD3P3_CPU), U1.43 (VDDA), U1.46 (VDDA), U1.9 (CHIP_PU), U2.3 (VOUT)
- no-connect marks 2 -> 27
Other:
- note added: "High: Chip On Low: Chip Off"
- note removed: "GND from ESP"
- note removed: "GPIO Inputs from ESP"
- note removed: "NOTE: Using ESP separate from this board. Connections will go to the pinouts,"
- moved on the sheet: D1, D10, D11, D12, D13, D14, D15, D16, D17, D18, D19, D2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
